Commit message: getting application environment setup

File: evd_ros_backend/evd_ros_tasks/tasks/3d_printer_machine_tending/application.urdf.xacro (robot description, xacro)
@@ -1,4 +1,5 @@
 <?xml version="1.0"?>
-<application name="application" xmlns:xacro="http://ros.org/wiki/xacro">
+<robot name="application" xmlns:xacro="http://ros.org/wiki/xacro">
+  <xacro:arg name="kinematics_config" default="$(find ur_e_description)/config/ur3e_default.yaml"/>
   <!-- Common -->
   <link name="world" />
@@ -10,5 +11,5 @@
   </joint>
   <!-- Robot -->
-  <xacro:include filename="$(find evd_ros_core)/description/robot.urdf.xacro'" />
+  <xacro:include filename="$(find evd_ros_core)/description/robot.urdf.xacro"/>
   <joint name="app_robot_common_joint" type="fixed">
     <parent link="app"/>
@@ -19,8 +20,14 @@
   <link name="table_link" type="fixed">
     <visual>
-      <mesh filename="package://evd_ros_tasks/tasks/3d_printer_machine_tending/Table/Table.stl"/>
+      <origin rpy="0 0 0" xyz="0 0 0"/>
+      <geometry>
+        <mesh filename="package://evd_ros_tasks/tasks/3d_printer_machine_tending/models/Table/Table.stl" scale="0.000001 0.000001 0.000001"/>
+      </geometry>
     </visual>
     <collision>
-      <mesh filename="package://evd_ros_tasks/tasks/3d_printer_machine_tending/Table/Table.stl"/>
+      <origin rpy="0 0 0" xyz="0 0 0"/>
+      <geometry>
+        <mesh filename="package://evd_ros_tasks/tasks/3d_printer_machine_tending/collision_meshes/Table.stl" scale="0.000001 0.000001 0.000001"/>
+      </geometry>
     </collision>
   </link>
@@ -33,8 +40,14 @@
   <link name="3d_printer_link" type="fixed">
     <visual>
-      <mesh filename="package://evd_ros_tasks/tasks/3d_printer_machine_tending/MK2-Printer/MK2-Printer.stl"/>
+      <origin rpy="0 0 0" xyz="0 0 0"/>
+      <geometry>
+        <mesh filename="package://evd_ros_tasks/tasks/3d_printer_machine_tending/models/MK2-Printer/MK2-Printer.stl" scale="0.001 0.001 0.001"/>
+      </geometry>
     </visual>
     <collision>
-      <mesh filename="package://evd_ros_tasks/tasks/3d_printer_machine_tending/MK2-Printer/MK2-Printer.stl"/>
+      <origin rpy="0 0 0" xyz="0 0 0"/>
+      <geometry>
+        <mesh filename="package://evd_ros_tasks/tasks/3d_printer_machine_tending/collision_meshes/MK2-Printer.stl" scale="0.000001 0.000001 0.000001"/>
+      </geometry>
     </collision>
   </link>
@@ -47,8 +60,14 @@
   <link name="box_link" type="fixed">
     <visual>
-      <mesh filename="package://evd_ros_tasks/tasks/3d_printer_machine_tending/Box/Box.stl"/>
+      <origin rpy="0 0 0" xyz="0 0 0"/>
+      <geometry>
+        <mesh filename="package://evd_ros_tasks/tasks/3d_printer_machine_tending/models/Box/Box.stl" scale="0.001 0.001 0.001"/>
+      </geometry>
     </visual>
     <collision>
-      <mesh filename="package://evd_ros_tasks/tasks/3d_printer_machine_tending/Box/Box.stl"/>
+      <origin rpy="0 0 0" xyz="0 0 0"/>
+      <geometry>
+        <mesh filename="package://evd_ros_tasks/tasks/3d_printer_machine_tending/collision_meshes/Box.stl" scale="0.001 0.001 0.001"/>
+      </geometry>
     </collision>
   </link>
@@ -61,8 +80,14 @@
   <link name="ur3e_pedestal_link" type="fixed" >
     <visual>
-      <mesh filename="package://evd_ros_tasks/tasks/3d_printer_machine_tending/ur3e-Pedestal/Pedestal.stl"/>
+      <origin rpy="0 0 0" xyz="0 0 0"/>
+      <geometry>
+        <mesh filename="package://evd_ros_tasks/tasks/3d_printer_machine_tending/models/ur3e-Pedestal/Pedestal.stl" scale="0.000001 0.000001 0.000001"/>
+      </geometry>
     </visual>
     <collision>
-      <mesh filename="package://evd_ros_tasks/tasks/3d_printer_machine_tending/ur3e-Pedestal/Pedestal.stl"/>
+      <origin rpy="0 0 0" xyz="0 0 0"/>
+      <geometry>
+        <mesh filename="package://evd_ros_tasks/tasks/3d_printer_machine_tending/collision_meshes/Pedestal.stl" scale="0.000001 0.000001 0.000001"/>
+      </geometry>
     </collision>
   </link>
@@ -72,3 +97,3 @@
     <origin xyz="0.0 0.0 0.0" rpy="0.0 0.0 0.0" />
   </joint>
-</application>
+</robot>

Commit message: updating box collision mesh, removing scalars from xacro

File: evd_ros_backend/evd_ros_tasks/tasks/3d_printer_machine_tending/application.urdf.xacro (robot description, xacro)
@@ -22,5 +22,5 @@
       <origin rpy="0 0 0" xyz="0 0 0"/>
       <geometry>
-        <mesh filename="package://evd_ros_tasks/tasks/3d_printer_machine_tending/models/Table/Table.stl" scale="0.000001 0.000001 0.000001"/>
+        <mesh filename="package://evd_ros_tasks/tasks/3d_printer_machine_tending/models/Table/Table.stl"/>
       </geometry>
     </visual>
@@ -28,5 +28,5 @@
       <origin rpy="0 0 0" xyz="0 0 0"/>
       <geometry>
-        <mesh filename="package://evd_ros_tasks/tasks/3d_printer_machine_tending/collision_meshes/Table.stl" scale="0.000001 0.000001 0.000001"/>
+        <mesh filename="package://evd_ros_tasks/tasks/3d_printer_machine_tending/collision_meshes/Table.stl"/>
       </geometry>
     </collision>
@@ -42,5 +42,5 @@
       <origin rpy="0 0 0" xyz="0 0 0"/>
       <geometry>
-        <mesh filename="package://evd_ros_tasks/tasks/3d_printer_machine_tending/models/MK2-Printer/MK2-Printer.stl" scale="0.001 0.001 0.001"/>
+        <mesh filename="package://evd_ros_tasks/tasks/3d_printer_machine_tending/models/MK2-Printer/MK2-Printer.stl"/>
       </geometry>
     </visual>
@@ -48,5 +48,5 @@
       <origin rpy="0 0 0" xyz="0 0 0"/>
       <geometry>
-        <mesh filename="package://evd_ros_tasks/tasks/3d_printer_machine_tending/collision_meshes/MK2-Printer.stl" scale="0.000001 0.000001 0.000001"/>
+        <mesh filename="package://evd_ros_tasks/tasks/3d_printer_machine_tending/collision_meshes/MK2-Printer.stl"/>
       </geometry>
     </collision>
@@ -62,5 +62,5 @@
       <origin rpy="0 0 0" xyz="0 0 0"/>
       <geometry>
-        <mesh filename="package://evd_ros_tasks/tasks/3d_printer_machine_tending/models/Box/Box.stl" scale="0.001 0.001 0.001"/>
+        <mesh filename="package://evd_ros_tasks/tasks/3d_printer_machine_tending/models/Box/Box.stl"/>
       </geometry>
     </visual>
@@ -68,5 +68,5 @@
       <origin rpy="0 0 0" xyz="0 0 0"/>
       <geometry>
-        <mesh filename="package://evd_ros_tasks/tasks/3d_printer_machine_tending/collision_meshes/Box.stl" scale="0.001 0.001 0.001"/>
+        <mesh filename="package://evd_ros_tasks/tasks/3d_printer_machine_tending/collision_meshes/Box.stl"/>
       </geometry>
     </collision>
@@ -82,5 +82,5 @@
       <origin rpy="0 0 0" xyz="0 0 0"/>
       <geometry>
-        <mesh filename="package://evd_ros_tasks/tasks/3d_printer_machine_tending/models/ur3e-Pedestal/Pedestal.stl" scale="0.000001 0.000001 0.000001"/>
+        <mesh filename="package://evd_ros_tasks/tasks/3d_printer_machine_tending/models/ur3e-Pedestal/Pedestal.stl"/>
       </geometry>
     </visual>
@@ -88,5 +88,5 @@
       <origin rpy="0 0 0" xyz="0 0 0"/>
       <geometry>
-        <mesh filename="package://evd_ros_tasks/tasks/3d_printer_machine_tending/collision_meshes/Pedestal.stl" scale="0.000001 0.000001 0.000001"/>
+        <mesh filename="package://evd_ros_tasks/tasks/3d_printer_machine_tending/collision_meshes/Pedestal.stl"/>
       </geometry>
     </collision>

Commit message: working on configuring application environment

File: evd_ros_backend/evd_ros_tasks/tasks/3d_printer_machine_tending/application.urdf.xacro (robot description, xacro)
@@ -2,4 +2,7 @@
 <robot name="application" xmlns:xacro="http://ros.org/wiki/xacro">
   <xacro:arg name="kinematics_config" default="$(find ur_e_description)/config/ur3e_default.yaml"/>
+  <material name="visual_app_mesh">
+    <color rgba="${128/255} ${128/255} ${128/255} 1.0"/>
+  </material>
   <!-- Common -->
   <link name="world" />
@@ -9,4 +12,24 @@
     <child link="app"/>
     <origin xyz="0.0 0.0 0.0" rpy="0.0 0.0 0.0" />
+  </joint>
+  <!-- Location Marker Test -->
+  <link name="location_marker_test_link" type="fixed">
+    <visual>
+      <origin rpy="0 0 0" xyz="0 0 0"/>
+      <geometry>
+        <mesh filename="package://evd_ros_core/markers/LocationMarker.stl"/>
+      </geometry>
+    </visual>
+    <collision>
+      <origin rpy="0 0 0" xyz="0 0 0"/>
+      <geometry>
+        <mesh filename="package://evd_ros_core/markers/LocationMarker.stl"/>
+      </geometry>
+    </collision>
+  </link>
+  <joint name="app_location_joint" type="fixed">
+    <parent link="app"/>
+    <child link="location_marker_test_link"/>
+    <origin xyz="0.0 1.0 0.0" rpy="0.0 0.0 0.0" />
   </joint>
   <!-- Robot -->
@@ -24,4 +47,5 @@
         <mesh filename="package://evd_ros_tasks/tasks/3d_printer_machine_tending/models/Table/Table.stl"/>
       </geometry>
+      <material name="visual_app_mesh"/>
     </visual>
     <collision>
@@ -35,5 +59,5 @@
     <parent link="app" />
     <child link="table_link" />
-    <origin xyz="0.0 0.0 0.0" rpy="0.0 0.0 0.0" />
+    <origin xyz="0.0 0.35 -0.37" rpy="0.0 0.0 0.0" />
   </joint>
   <!-- 3D Printer -->
@@ -44,4 +68,5 @@
         <mesh filename="package://evd_ros_tasks/tasks/3d_printer_machine_tending/models/MK2-Printer/MK2-Printer.stl"/>
       </geometry>
+      <material name="visual_app_mesh"/>
     </visual>
     <collision>
@@ -55,5 +80,5 @@
     <parent link="app" />
     <child link="3d_printer_link" />
-    <origin xyz="0.0 0.0 0.0" rpy="0.0 0.0 0.0" />
+    <origin xyz="-0.28 0.32 0.3" rpy="0.0 0.0 0.0" />
   </joint>
   <!-- Product Box -->
@@ -64,4 +89,5 @@
         <mesh filename="package://evd_ros_tasks/tasks/3d_printer_machine_tending/models/Box/Box.stl"/>
       </geometry>
+      <material name="visual_app_mesh"/>
     </visual>
     <collision>
@@ -75,5 +101,5 @@
     <parent link="app" />
     <child link="box_link" />
-    <origin xyz="0.0 0.0 0.0" rpy="0.0 0.0 0.0" />
+    <origin xyz="0.35 0.35 0.07" rpy="0.0 0.0 0.0" />
   </joint>
   <!-- Robot Pedestal -->
@@ -84,4 +110,5 @@
         <mesh filename="package://evd_ros_tasks/tasks/3d_printer_machine_tending/models/ur3e-Pedestal/Pedestal.stl"/>
       </geometry>
+      <material name="visual_app_mesh"/>
     </visual>
     <collision>
@@ -95,5 +122,5 @@
     <parent link="robot_common" />
     <child link="ur3e_pedestal_link" />
-    <origin xyz="0.0 0.0 0.0" rpy="0.0 0.0 0.0" />
+    <origin xyz="0.0 0.0 -0.38" rpy="0.0 0.0 0.0" />
   </joint>
 </robot>

Commit message: removing location marker from application xacro

File: evd_ros_backend/evd_ros_tasks/tasks/3d_printer_machine_tending/application.urdf.xacro (robot description, xacro)
@@ -12,24 +12,4 @@
     <child link="app"/>
     <origin xyz="0.0 0.0 0.0" rpy="0.0 0.0 0.0" />
-  </joint>
-  <!-- Location Marker Test -->
-  <link name="location_marker_test_link" type="fixed">
-    <visual>
-      <origin rpy="0 0 0" xyz="0 0 0"/>
-      <geometry>
-        <mesh filename="package://evd_ros_core/markers/LocationMarker.stl"/>
-      </geometry>
-    </visual>
-    <collision>
-      <origin rpy="0 0 0" xyz="0 0 0"/>
-      <geometry>
-        <mesh filename="package://evd_ros_core/markers/LocationMarker.stl"/>
-      </geometry>
-    </collision>
-  </link>
-  <joint name="app_location_joint" type="fixed">
-    <parent link="app"/>
-    <child link="location_marker_test_link"/>
-    <origin xyz="0.0 1.0 0.0" rpy="0.0 0.0 0.0" />
   </joint>
   <!-- Robot -->

Commit message: waypoints converted to living within the context instead of a trajectory

File: evd_ros_backend/evd_ros_tasks/tasks/3d_printer_machine_tending/application.urdf.xacro (robot description, xacro)
@@ -39,5 +39,5 @@
     <parent link="app" />
     <child link="table_link" />
-    <origin xyz="0.0 0.35 -0.37" rpy="0.0 0.0 0.0" />
+    <origin xyz="0.0 0.36 -0.37" rpy="0.0 0.0 0.0" />
   </joint>
   <!-- 3D Printer -->
