Commit message: pybullet simulation now actually moving properly - need to tune parameters, hook in interpolator, and extract collision state

File: evd_ros_backend/evd_ros_tasks/config/pybullet/model.urdf (robot description, URDF)
Before this commit: robot planner_ur3e_robotiq_85_pluw_workcell, 25 links, 24 joints
Links:
- removed link planner_base
- removed link planner_base_link
- removed link planner_ee_link
- removed link planner_forearm_link
- removed link planner_robotiq_85_base_link
- removed link planner_robotiq_85_left_finger_link
- removed link planner_robotiq_85_left_finger_tip_link
- removed link planner_robotiq_85_left_inner_knuckle_link
- removed link planner_robotiq_85_left_knuckle_link
- removed link planner_robotiq_85_right_finger_link
- removed link planner_robotiq_85_right_finger_tip_link
- removed link planner_robotiq_85_right_inner_knuckle_link
- removed link planner_robotiq_85_right_knuckle_link
- removed link planner_shoulder_link
- removed link planner_tool0
- removed link planner_upper_arm_link
- removed link planner_wrist_1_link
- removed link planner_wrist_2_link
- removed link planner_wrist_3_link
- added link base
- added link base_link, mass 2.0; collision mesh filename=./meshes/collision/base.stl; visual mesh filename=./meshes/visual/base.dae
- added link ee_link; collision box size=0.01 0.01 0.01
- added link forearm_link, mass 1.26; collision mesh filename=./meshes/collision/forearm.stl; visual mesh filename=./meshes/visual/forearm.dae
- added link robotiq_85_base_link, mass 0.636951; collision mesh filename=./meshes/collision/robotiq_85_base_link.stl; visual mesh filename=./meshes/visual/robotiq_85_base_link.dae
- added link robotiq_85_left_finger_link, mass 0.027309; collision mesh filename=./meshes/collision/robotiq_85_finger_link.stl; visual mesh filename=./meshes/visual/robotiq_85_finger_link.dae
- added link robotiq_85_left_finger_tip_link, mass 0.019555; collision mesh filename=./meshes/collision/robotiq_85_finger_tip_link.stl; visual mesh filename=./meshes/visual/robotiq_85_finger_tip_link.dae
- added link robotiq_85_left_inner_knuckle_link, mass 0.029951; collision mesh filename=./meshes/collision/robotiq_85_inner_knuckle_link.stl; visual mesh filename=./meshes/visual/robotiq_85_inner_knuckle_link.dae
- added link robotiq_85_left_knuckle_link, mass 0.018491; collision mesh filename=./meshes/collision/robotiq_85_knuckle_link.stl; visual mesh filename=./meshes/visual/robotiq_85_knuckle_link.dae
- added link robotiq_85_right_finger_link, mass 0.027309; collision mesh filename=./meshes/collision/robotiq_85_finger_link.stl; visual mesh filename=./meshes/visual/robotiq_85_finger_link.dae
- added link robotiq_85_right_finger_tip_link, mass 0.019555; collision mesh filename=./meshes/collision/robotiq_85_finger_tip_link.stl; visual mesh filename=./meshes/visual/robotiq_85_finger_tip_link.dae
- added link robotiq_85_right_inner_knuckle_link, mass 0.029951; collision mesh filename=./meshes/collision/robotiq_85_inner_knuckle_link.stl; visual mesh filename=./meshes/visual/robotiq_85_inner_knuckle_link.dae
- added link robotiq_85_right_knuckle_link, mass 0.018491; collision mesh filename=./meshes/collision/robotiq_85_knuckle_link.stl; visual mesh filename=./meshes/visual/robotiq_85_knuckle_link.dae
- added link shoulder_link, mass 2.0; collision mesh filename=./meshes/collision/shoulder.stl; visual mesh filename=./meshes/visual/shoulder.dae
- added link tool0
- added link upper_arm_link, mass 3.42; collision mesh filename=./meshes/collision/upperarm.stl; visual mesh filename=./meshes/visual/upperarm.dae
- added link wrist_1_link, mass 0.8; collision mesh filename=./meshes/collision/wrist1.stl; visual mesh filename=./meshes/visual/wrist1.dae
- added link wrist_2_link, mass 0.8; collision mesh filename=./meshes/collision/wrist2.stl; visual mesh filename=./meshes/visual/wrist2.dae
- added link wrist_3_link, mass 0.35; collision mesh filename=./meshes/collision/wrist3.stl; visual mesh filename=./meshes/visual/wrist3.dae
Joints:
- removed joint planner_base_link-base_fixed_joint
- removed joint planner_ee_fixed_joint
- removed joint planner_elbow_joint
- removed joint planner_robotiq_85_base_joint
- removed joint planner_robotiq_85_left_finger_joint
- removed joint planner_robotiq_85_left_finger_tip_joint
- removed joint planner_robotiq_85_left_inner_knuckle_joint
- removed joint planner_robotiq_85_left_knuckle_joint
- removed joint planner_robotiq_85_right_finger_joint
- removed joint planner_robotiq_85_right_finger_tip_joint
- removed joint planner_robotiq_85_right_inner_knuckle_joint
- removed joint planner_robotiq_85_right_knuckle_joint
- removed joint planner_shoulder_lift_joint
- removed joint planner_shoulder_pan_joint
- removed joint planner_wrist_1_joint
- removed joint planner_wrist_2_joint
- removed joint planner_wrist_3_joint
- removed joint planner_wrist_3_link-tool0_fixed_joint
- added joint base_link-base_fixed_joint: type fixed, parent base_link, child base, origin xyz=0 0 0 rpy=0 0 -3.14159265359
- added joint ee_fixed_joint: type fixed, parent wrist_3_link, child ee_link, origin xyz=0.0 0.092 0.0 rpy=0.0 0.0 1.57079632679
- added joint elbow_joint: type revolute, parent upper_arm_link, child forearm_link, origin xyz=0.0 -0.093 0.244 rpy=0.0 0.0 0.0, axis 0 1 0, limit lower=-3.14159265359 upper=3.14159265359 effort=150.0 velocity=3.14
- added joint robotiq_85_base_joint: type fixed, parent tool0, child robotiq_85_base_link, origin xyz=0 0 0 rpy=1.570795 -1.570795 0
- added joint robotiq_85_left_finger_joint: type continuous, parent robotiq_85_left_knuckle_link, child robotiq_85_left_finger_link, origin xyz=-0.00408552455 -0.03148604435 0.0 rpy=0 0 0
- added joint robotiq_85_left_finger_tip_joint: type continuous, parent robotiq_85_left_inner_knuckle_link, child robotiq_85_left_finger_tip_link, origin xyz=0.04303959807 -0.03759940821 0.0 rpy=0.0 0.0 0.0, axis 0 0 1, limit lower=-3.14 upper=3.14 effort=0.1 velocity=100.0, mimic joint=robotiq_85_left_knuckle_joint multiplier=-1
- added joint robotiq_85_left_inner_knuckle_joint: type continuous, parent robotiq_85_base_link, child robotiq_85_left_inner_knuckle_link, origin xyz=0.06142 0.0127 0 rpy=3.14159 0.0 0.0, axis 0 0 1, limit lower=-3.14 upper=3.14 effort=0.1 velocity=100.0, mimic joint=robotiq_85_left_knuckle_joint offset=0
- added joint robotiq_85_left_knuckle_joint: type revolute, parent robotiq_85_base_link, child robotiq_85_left_knuckle_link, origin xyz=0.05490451627 0.03060114443 0.0 rpy=3.14159 0.0 0.0, axis 0 0 1, limit lower=0.0 upper=0.804 effort=1000 velocity=2.0
- added joint robotiq_85_right_finger_joint: type continuous, parent robotiq_85_right_knuckle_link, child robotiq_85_right_finger_link, origin xyz=-0.00408552455 -0.03148604435 0.0 rpy=0 0 0
- added joint robotiq_85_right_finger_tip_joint: type continuous, parent robotiq_85_right_inner_knuckle_link, child robotiq_85_right_finger_tip_link, origin xyz=0.04303959807 -0.03759940821  0.0 rpy=0.0 0.0 0.0, axis 0 0 1, limit lower=-3.14 upper=3.14 effort=0.1 velocity=100.0, mimic joint=robotiq_85_left_knuckle_joint multiplier=-1
- added joint robotiq_85_right_inner_knuckle_joint: type continuous, parent robotiq_85_base_link, child robotiq_85_right_inner_knuckle_link, origin xyz=0.06142 -0.0127 0 rpy=0 0 0, axis 0 0 1, limit lower=-3.14 upper=3.14 effort=0.1 velocity=100.0, mimic joint=robotiq_85_left_knuckle_joint offset=0
- added joint robotiq_85_right_knuckle_joint: type continuous, parent robotiq_85_base_link, child robotiq_85_right_knuckle_link, origin xyz=0.05490451627 -0.03060114443 0.0 rpy=0.0 0.0 0.0, axis 0 0 1, limit lower=-3.14 upper=3.14 effort=1000 velocity=100.0, mimic joint=robotiq_85_left_knuckle_joint
- added joint shoulder_lift_joint: type revolute, parent shoulder_link, child upper_arm_link, origin xyz=0.0 0.12 0.0 rpy=0.0 1.57079632679 0.0, axis 0 1 0, limit lower=-6.28318530718 upper=6.28318530718 effort=330.0 velocity=3.14
- added joint shoulder_pan_joint: type revolute, parent base_link, child shoulder_link, origin xyz=0.0 0.0 0.152 rpy=0.0 0.0 0.0, axis 0 0 1, limit lower=-6.28318530718 upper=6.28318530718 effort=330.0 velocity=3.14
- added joint wrist_1_joint: type revolute, parent forearm_link, child wrist_1_link, origin xyz=0.0 0.0 0.213 rpy=0.0 1.57079632679 0.0, axis 0 1 0, limit lower=-6.28318530718 upper=6.28318530718 effort=54.0 velocity=6.28
- added joint wrist_2_joint: type revolute, parent wrist_1_link, child wrist_2_link, origin xyz=0.0 0.104 0.0 rpy=0.0 0.0 0.0, axis 0 0 1, limit lower=-6.28318530718 upper=6.28318530718 effort=54.0 velocity=6.28
- added joint wrist_3_joint: type revolute, parent wrist_2_link, child wrist_3_link, origin xyz=0.0 0.0 0.085 rpy=0.0 0.0 0.0, axis 0 1 0, limit lower=-6.28318530718 upper=6.28318530718 effort=54.0 velocity=6.28
- added joint wrist_3_link-tool0_fixed_joint: type fixed, parent wrist_3_link, child tool0, origin xyz=0 0.092 0 rpy=-1.57079632679 0 0
- joint robot_common_ur3e_pedestal_joint: parent planner_base_link -> base_link
- joint world_baselink_joint: child planner_base_link -> base_link
