Commit message: fixing urdfs

File: evd_ros_backend/evd_ros_tasks/config/pybullet/environment.urdf (robot description, URDF)
Before this commit: robot environment, 4 links, 2 joints
Links:
- added link blade_conveyor_link; collision mesh filename=./environment/collision/conveyor.stl; visual mesh filename=./environment/visual/conveyor.stl
- added link blade_feeder_link; collision mesh filename=./environment/collision/blade_feeder.stl; visual mesh filename=./environment/visual/blade_feeder.stl
- added link knife_conveyor_link; collision mesh filename=./environment/collision/conveyor.stl; visual mesh filename=./environment/visual/conveyor.stl
- added link knife_feeder_link; collision mesh filename=./environment/collision/knife_feeder.stl; visual mesh filename=./environment/visual/knife_feeder.stl
- link 3d_printer_link: geometry collision mesh filename=./environment/collision/MK2-Printer.stl; visual mesh filename=./environment/visual/MK2-Printer.stl
- link assembly_jig_link: geometry collision mesh filename=./environment/collision/assembly_jig.stl; visual mesh filename=./environment/visual/assembly_jig.stl
- link table_link: geometry collision mesh filename=./environment/collision/Table.stl; visual mesh filename=./environment/visual/Table.stl
Joints:
- added joint env_assembly_jig_joint: type fixed, parent env_base, child assembly_jig_link, origin xyz=-0.28 0.32 0.3 rpy=0.0 0.0 0.0
- added joint env_blade_conveyor_joint: type fixed, parent env_base, child blade_conveyor_link, origin xyz=-0.28 0.32 0.3 rpy=0.0 0.0 0.0
- added joint env_blade_feeder_joint: type fixed, parent env_base, child blade_feeder_link, origin xyz=-0.28 0.32 0.3 rpy=0.0 0.0 0.0
- added joint env_knife_conveyor_joint: type fixed, parent env_base, child knife_conveyor_link, origin xyz=-0.28 0.32 0.3 rpy=0.0 0.0 0.0
- added joint env_knife_feeder_joint: type fixed, parent env_base, child knife_feeder_link, origin xyz=-0.28 0.32 0.3 rpy=0.0 0.0 0.0
- joint env_3d_printer_joint: child assembly_jig_link -> 3d_printer_link

File: evd_ros_backend/evd_ros_tasks/config/pybullet/robot.urdf (robot description, URDF)
Before this commit: robot robot, 62 links, 61 joints
Links:
- link physical_base_link_inertia: geometry collision mesh filename=./robot/collision/base.stl; visual mesh filename=./robot/visual/base.dae
- link physical_forearm_link: geometry collision mesh filename=./robot/collision/forearm.stl; visual mesh filename=./robot/visual/forearm.dae
- link physical_robotiq_85_base_link: geometry collision mesh filename=./robot/collision/robotiq_85_base_link.stl; visual mesh filename=./robot/visual/robotiq_85_base_link.dae
- link physical_robotiq_85_left_finger_link: geometry collision mesh filename=./robot/collision/robotiq_85_finger_link.stl; visual mesh filename=./robot/visual/robotiq_85_finger_link.dae
- link physical_robotiq_85_left_finger_tip_link: geometry collision mesh filename=./robot/collision/robotiq_85_finger_tip_link.stl; visual mesh filename=./robot/visual/robotiq_85_finger_tip_link.dae
- link physical_robotiq_85_left_inner_knuckle_link: geometry collision mesh filename=./robot/collision/robotiq_85_inner_knuckle_link.stl; visual mesh filename=./robot/visual/robotiq_85_inner_knuckle_link.dae
- link physical_robotiq_85_left_knuckle_link: geometry collision mesh filename=./robot/collision/robotiq_85_knuckle_link.stl; visual mesh filename=./robot/visual/robotiq_85_knuckle_link.dae
- link physical_robotiq_85_right_finger_link: geometry collision mesh filename=./robot/collision/robotiq_85_finger_link.stl; visual mesh filename=./robot/visual/robotiq_85_finger_link.dae
- link physical_robotiq_85_right_finger_tip_link: geometry collision mesh filename=./robot/collision/robotiq_85_finger_tip_link.stl; visual mesh filename=./robot/visual/robotiq_85_finger_tip_link.dae
- link physical_robotiq_85_right_inner_knuckle_link: geometry collision mesh filename=./robot/collision/robotiq_85_inner_knuckle_link.stl; visual mesh filename=./robot/visual/robotiq_85_inner_knuckle_link.dae
- link physical_robotiq_85_right_knuckle_link: geometry collision mesh filename=./robot/collision/robotiq_85_knuckle_link.stl; visual mesh filename=./robot/visual/robotiq_85_knuckle_link.dae
- link physical_shoulder_link: geometry collision mesh filename=./robot/collision/shoulder.stl; visual mesh filename=./robot/visual/shoulder.dae
- link physical_upper_arm_link: geometry collision mesh filename=./robot/collision/upperarm.stl; visual mesh filename=./robot/visual/upperarm.dae
- link physical_wrist_1_link: geometry collision mesh filename=./robot/collision/wrist1.stl; visual mesh filename=./robot/visual/wrist1.dae
- link physical_wrist_2_link: geometry collision mesh filename=./robot/collision/wrist2.stl; visual mesh filename=./robot/visual/wrist2.dae
- link physical_wrist_3_link: geometry collision mesh filename=./robot/collision/wrist3.stl; visual mesh filename=./robot/visual/wrist3.dae
- link planner_base_link_inertia: geometry collision mesh filename=./robot/collision/base.stl; visual mesh filename=./robot/visual/base.dae
- link planner_forearm_link: geometry collision mesh filename=./robot/collision/forearm.stl; visual mesh filename=./robot/visual/forearm.dae
- link planner_robotiq_85_base_link: geometry collision mesh filename=./robot/collision/robotiq_85_base_link.stl; visual mesh filename=./robot/visual/robotiq_85_base_link.dae
- link planner_robotiq_85_left_finger_link: geometry collision mesh filename=./robot/collision/robotiq_85_finger_link.stl; visual mesh filename=./robot/visual/robotiq_85_finger_link.dae
- link planner_robotiq_85_left_finger_tip_link: geometry collision mesh filename=./robot/collision/robotiq_85_finger_tip_link.stl; visual mesh filename=./robot/visual/robotiq_85_finger_tip_link.dae
- link planner_robotiq_85_left_inner_knuckle_link: geometry collision mesh filename=./robot/collision/robotiq_85_inner_knuckle_link.stl; visual mesh filename=./robot/visual/robotiq_85_inner_knuckle_link.dae
- link planner_robotiq_85_left_knuckle_link: geometry collision mesh filename=./robot/collision/robotiq_85_knuckle_link.stl; visual mesh filename=./robot/visual/robotiq_85_knuckle_link.dae
- link planner_robotiq_85_right_finger_link: geometry collision mesh filename=./robot/collision/robotiq_85_finger_link.stl; visual mesh filename=./robot/visual/robotiq_85_finger_link.dae
- link planner_robotiq_85_right_finger_tip_link: geometry collision mesh filename=./robot/collision/robotiq_85_finger_tip_link.stl; visual mesh filename=./robot/visual/robotiq_85_finger_tip_link.dae
- link planner_robotiq_85_right_inner_knuckle_link: geometry collision mesh filename=./robot/collision/robotiq_85_inner_knuckle_link.stl; visual mesh filename=./robot/visual/robotiq_85_inner_knuckle_link.dae
- link planner_robotiq_85_right_knuckle_link: geometry collision mesh filename=./robot/collision/robotiq_85_knuckle_link.stl; visual mesh filename=./robot/visual/robotiq_85_knuckle_link.dae
- link planner_shoulder_link: geometry collision mesh filename=./robot/collision/shoulder.stl; visual mesh filename=./robot/visual/shoulder.dae
- link planner_upper_arm_link: geometry collision mesh filename=./robot/collision/upperarm.stl; visual mesh filename=./robot/visual/upperarm.dae
- link planner_wrist_1_link: geometry collision mesh filename=./robot/collision/wrist1.stl; visual mesh filename=./robot/visual/wrist1.dae
- link planner_wrist_2_link: geometry collision mesh filename=./robot/collision/wrist2.stl; visual mesh filename=./robot/visual/wrist2.dae
- link planner_wrist_3_link: geometry collision mesh filename=./robot/collision/wrist3.stl; visual mesh filename=./robot/visual/wrist3.dae
- link simulated_base_link_inertia: geometry collision mesh filename=./robot/collision/base.stl; visual mesh filename=./robot/visual/base.dae
- link simulated_forearm_link: geometry collision mesh filename=./robot/collision/forearm.stl; visual mesh filename=./robot/visual/forearm.dae
- link simulated_robotiq_85_base_link: geometry collision mesh filename=./robot/collision/robotiq_85_base_link.stl; visual mesh filename=./robot/visual/robotiq_85_base_link.dae
- link simulated_robotiq_85_left_finger_link: geometry collision mesh filename=./robot/collision/robotiq_85_finger_link.stl; visual mesh filename=./robot/visual/robotiq_85_finger_link.dae
- link simulated_robotiq_85_left_finger_tip_link: geometry collision mesh filename=./robot/collision/robotiq_85_finger_tip_link.stl; visual mesh filename=./robot/visual/robotiq_85_finger_tip_link.dae
- link simulated_robotiq_85_left_inner_knuckle_link: geometry collision mesh filename=./robot/collision/robotiq_85_inner_knuckle_link.stl; visual mesh filename=./robot/visual/robotiq_85_inner_knuckle_link.dae
- link simulated_robotiq_85_left_knuckle_link: geometry collision mesh filename=./robot/collision/robotiq_85_knuckle_link.stl; visual mesh filename=./robot/visual/robotiq_85_knuckle_link.dae
- link simulated_robotiq_85_right_finger_link: geometry collision mesh filename=./robot/collision/robotiq_85_finger_link.stl; visual mesh filename=./robot/visual/robotiq_85_finger_link.dae
- link simulated_robotiq_85_right_finger_tip_link: geometry collision mesh filename=./robot/collision/robotiq_85_finger_tip_link.stl; visual mesh filename=./robot/visual/robotiq_85_finger_tip_link.dae
- link simulated_robotiq_85_right_inner_knuckle_link: geometry collision mesh filename=./robot/collision/robotiq_85_inner_knuckle_link.stl; visual mesh filename=./robot/visual/robotiq_85_inner_knuckle_link.dae
- link simulated_robotiq_85_right_knuckle_link: geometry collision mesh filename=./robot/collision/robotiq_85_knuckle_link.stl; visual mesh filename=./robot/visual/robotiq_85_knuckle_link.dae
- link simulated_shoulder_link: geometry collision mesh filename=./robot/collision/shoulder.stl; visual mesh filename=./robot/visual/shoulder.dae
- link simulated_upper_arm_link: geometry collision mesh filename=./robot/collision/upperarm.stl; visual mesh filename=./robot/visual/upperarm.dae
- link simulated_wrist_1_link: geometry collision mesh filename=./robot/collision/wrist1.stl; visual mesh filename=./robot/visual/wrist1.dae
- link simulated_wrist_2_link: geometry collision mesh filename=./robot/collision/wrist2.stl; visual mesh filename=./robot/visual/wrist2.dae
- link simulated_wrist_3_link: geometry collision mesh filename=./robot/collision/wrist3.stl; visual mesh filename=./robot/visual/wrist3.dae

File: evd_ros_backend/evd_ros_tasks/description/ur3e.urdf.xacro (robot description, xacro)
@@ -2,4 +2,7 @@
 <robot name="robot" xmlns:xacro="http://ros.org/wiki/xacro">
 	<xacro:arg name="kinematics_config" default="$(find ur_description)/config/ur3e_default.yaml"/>
+	<material name="visual_env_mesh">
+		<color rgba="${128/255} ${128/255} ${128/255} 1.0"/>
+	</material>
 	<!-- robot_common -->
 	<link name="robot_common" />
@@ -53,5 +56,5 @@
         <mesh filename="package://evd_ros_tasks/description/meshes/visual/Pedestal.stl"/>
       </geometry>
-      <material name="visual_app_mesh"/>
+      <material name="visual_env_mesh"/>
     </visual>
     <collision>
