Commit message: tweaking pybullet model + pybullet variant of URDF

File: evd_ros_backend/evd_ros_tasks/config/pybullet/environment.urdf (robot description, URDF)
Before this commit: robot environment, 8 links, 7 joints
Links:
- link 3d_printer_link: geometry visual mesh filename=./environment/visual/MK2-Printer.stl
- link assembly_jig_link: geometry visual mesh filename=./environment/visual/assembly_jig.stl
- link blade_conveyor_link: geometry visual mesh filename=./environment/visual/conveyor.stl
- link blade_feeder_link: geometry visual mesh filename=./environment/visual/blade_feeder.stl
- link knife_conveyor_link: geometry visual mesh filename=./environment/visual/conveyor.stl
- link knife_feeder_link: geometry visual mesh filename=./environment/visual/knife_feeder.stl
- link table_link: geometry visual mesh filename=./environment/visual/Table.stl
Joints:
- joint env_assembly_jig_joint: origin xyz=-0.28 0.32 0.3 rpy=0.0 0.0 0.0 -> xyz=0.2 0.28 0.14 rpy=0.0 1.5707963 1.5707963
- joint env_blade_conveyor_joint: origin xyz=-0.28 0.32 0.3 rpy=0.0 0.0 0.0 -> xyz=-0.85 -0.25 -0.75 rpy=0.0 0.0 1.5707963
- joint env_blade_feeder_joint: origin xyz=-0.28 0.32 0.3 rpy=0.0 0.0 0.0 -> xyz=-0.85 -0.25 -0.75 rpy=0.0 0.0 1.5707963
- joint env_knife_conveyor_joint: origin xyz=-0.28 0.32 0.3 rpy=0.0 0.0 0.0 -> xyz=0.85 -0.25 -0.75 rpy=0.0 0.0 -1.5707963
- joint env_knife_feeder_joint: origin xyz=-0.28 0.32 0.3 rpy=0.0 0.0 0.0 -> xyz=0.85 -0.25 -0.75 rpy=0.0 0.0 -1.5707963

File: evd_ros_backend/evd_ros_tasks/config/pybullet/robot.urdf (robot description, URDF)
Before this commit: robot robot, 62 links, 61 joints
Links:
- removed link physical_base
- removed link physical_base_link
- removed link physical_base_link_inertia
- removed link physical_flange
- removed link physical_forearm_link
- removed link physical_robotiq_85_base_link
- removed link physical_robotiq_85_left_finger_link
- removed link physical_robotiq_85_left_finger_tip_link
- removed link physical_robotiq_85_left_inner_knuckle_link
- removed link physical_robotiq_85_left_knuckle_link
- removed link physical_robotiq_85_right_finger_link
- removed link physical_robotiq_85_right_finger_tip_link
- removed link physical_robotiq_85_right_inner_knuckle_link
- removed link physical_robotiq_85_right_knuckle_link
- removed link physical_shoulder_link
- removed link physical_tool0
- removed link physical_upper_arm_link
- removed link physical_wrist_1_link
- removed link physical_wrist_2_link
- removed link physical_wrist_3_link
- removed link planner_base
- removed link planner_base_link
- removed link planner_base_link_inertia
- removed link planner_flange
- removed link planner_forearm_link
- removed link planner_robotiq_85_base_link
- removed link planner_robotiq_85_left_finger_link
- removed link planner_robotiq_85_left_finger_tip_link
- removed link planner_robotiq_85_left_inner_knuckle_link
- removed link planner_robotiq_85_left_knuckle_link
- removed link planner_robotiq_85_right_finger_link
- removed link planner_robotiq_85_right_finger_tip_link
- removed link planner_robotiq_85_right_inner_knuckle_link
- removed link planner_robotiq_85_right_knuckle_link
- removed link planner_shoulder_link
- removed link planner_tool0
- removed link planner_upper_arm_link
- removed link planner_wrist_1_link
- removed link planner_wrist_2_link
- removed link planner_wrist_3_link
- removed link simulated_base
- removed link simulated_base_link
- removed link simulated_base_link_inertia
- removed link simulated_flange
- removed link simulated_forearm_link
- removed link simulated_robotiq_85_base_link
- removed link simulated_robotiq_85_left_finger_link
- removed link simulated_robotiq_85_left_finger_tip_link
- removed link simulated_robotiq_85_left_inner_knuckle_link
- removed link simulated_robotiq_85_left_knuckle_link
- removed link simulated_robotiq_85_right_finger_link
- removed link simulated_robotiq_85_right_finger_tip_link
- removed link simulated_robotiq_85_right_inner_knuckle_link
- removed link simulated_robotiq_85_right_knuckle_link
- removed link simulated_shoulder_link
- removed link simulated_tool0
- removed link simulated_upper_arm_link
- removed link simulated_wrist_1_link
- removed link simulated_wrist_2_link
- removed link simulated_wrist_3_link
- added link base
- added link base_link
- added link base_link_inertia, mass 2.0; visual mesh filename=./robot/visual/base.dae
- added link flange
- added link forearm_link, mass 1.26; visual mesh filename=./robot/visual/forearm.dae
- added link robotiq_85_base_link, mass 0.636951; visual mesh filename=./robot/visual/robotiq_85_base_link.dae
- added link robotiq_85_left_finger_link, mass 0.027309; visual mesh filename=./robot/visual/robotiq_85_finger_link.dae
- added link robotiq_85_left_finger_tip_link, mass 0.019555; visual mesh filename=./robot/visual/robotiq_85_finger_tip_link.dae
- added link robotiq_85_left_inner_knuckle_link, mass 0.029951; visual mesh filename=./robot/visual/robotiq_85_inner_knuckle_link.dae
- added link robotiq_85_left_knuckle_link, mass 0.018491; visual mesh filename=./robot/visual/robotiq_85_knuckle_link.dae
- added link robotiq_85_right_finger_link, mass 0.027309; visual mesh filename=./robot/visual/robotiq_85_finger_link.dae
- added link robotiq_85_right_finger_tip_link, mass 0.019555; visual mesh filename=./robot/visual/robotiq_85_finger_tip_link.dae
- added link robotiq_85_right_inner_knuckle_link, mass 0.029951; visual mesh filename=./robot/visual/robotiq_85_inner_knuckle_link.dae
- added link robotiq_85_right_knuckle_link, mass 0.018491; visual mesh filename=./robot/visual/robotiq_85_knuckle_link.dae
- added link shoulder_link, mass 2.0; visual mesh filename=./robot/visual/shoulder.dae
- added link tool0
- added link upper_arm_link, mass 3.42; visual mesh filename=./robot/visual/upperarm.dae
- added link wrist_1_link, mass 0.8; visual mesh filename=./robot/visual/wrist1.dae
- added link wrist_2_link, mass 0.8; visual mesh filename=./robot/visual/wrist2.dae
- added link wrist_3_link, mass 0.35; visual mesh filename=./robot/visual/wrist3.dae
- link ur3e_pedestal_link: geometry visual mesh filename=package://evd_ros_tasks/description/meshes/visual/Pedestal.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
Joints:
- removed joint physical_base_link-base_fixed_joint
- removed joint physical_base_link-base_link_inertia
- removed joint physical_common_joint
- removed joint physical_elbow_joint
- removed joint physical_flange-tool0
- removed joint physical_robotiq_85_base_joint
- removed joint physical_robotiq_85_left_finger_joint
- removed joint physical_robotiq_85_left_finger_tip_joint
- removed joint physical_robotiq_85_left_inner_knuckle_joint
- removed joint physical_robotiq_85_left_knuckle_joint
- removed joint physical_robotiq_85_right_finger_joint
- removed joint physical_robotiq_85_right_finger_tip_joint
- removed joint physical_robotiq_85_right_inner_knuckle_joint
- removed joint physical_robotiq_85_right_knuckle_joint
- removed joint physical_shoulder_lift_joint
- removed joint physical_shoulder_pan_joint
- removed joint physical_wrist_1_joint
- removed joint physical_wrist_2_joint
- removed joint physical_wrist_3-flange
- removed joint physical_wrist_3_joint
- removed joint planner_base_link-base_fixed_joint
- removed joint planner_base_link-base_link_inertia
- removed joint planner_elbow_joint
- removed joint planner_flange-tool0
- removed joint planner_robotiq_85_base_joint
- removed joint planner_robotiq_85_left_finger_joint
- removed joint planner_robotiq_85_left_finger_tip_joint
- removed joint planner_robotiq_85_left_inner_knuckle_joint
- removed joint planner_robotiq_85_left_knuckle_joint
- removed joint planner_robotiq_85_right_finger_joint
- removed joint planner_robotiq_85_right_finger_tip_joint
- removed joint planner_robotiq_85_right_inner_knuckle_joint
- removed joint planner_robotiq_85_right_knuckle_joint
- removed joint planner_shoulder_lift_joint
- removed joint planner_shoulder_pan_joint
- removed joint planner_world_joint
- removed joint planner_wrist_1_joint
- removed joint planner_wrist_2_joint
- removed joint planner_wrist_3-flange
- removed joint planner_wrist_3_joint
- removed joint simulated_base_link-base_fixed_joint
- removed joint simulated_base_link-base_link_inertia
- removed joint simulated_common_joint
- removed joint simulated_elbow_joint
- removed joint simulated_flange-tool0
- removed joint simulated_robotiq_85_base_joint
- removed joint simulated_robotiq_85_left_finger_joint
- removed joint simulated_robotiq_85_left_finger_tip_joint
- removed joint simulated_robotiq_85_left_inner_knuckle_joint
- removed joint simulated_robotiq_85_left_knuckle_joint
- removed joint simulated_robotiq_85_right_finger_joint
- removed joint simulated_robotiq_85_right_finger_tip_joint
- removed joint simulated_robotiq_85_right_inner_knuckle_joint
- removed joint simulated_robotiq_85_right_knuckle_joint
- removed joint simulated_shoulder_lift_joint
- removed joint simulated_shoulder_pan_joint
- removed joint simulated_wrist_1_joint
- removed joint simulated_wrist_2_joint
- removed joint simulated_wrist_3-flange
- removed joint simulated_wrist_3_joint
- added joint base_link-base_fixed_joint: type fixed, parent base_link, child base, origin xyz=0 0 0 rpy=0 0 3.141592653589793
- added joint base_link-base_link_inertia: type fixed, parent base_link, child base_link_inertia, origin xyz=0 0 0 rpy=0 0 3.141592653589793
- added joint elbow_joint: type revolute, parent upper_arm_link, child forearm_link, origin xyz=-0.24355 0 0 rpy=0 0 0, axis 0 0 1, limit lower=-3.141592653589793 upper=3.141592653589793 effort=28.0 velocity=3.141592653589793
- added joint flange-tool0: type fixed, parent flange, child tool0, origin xyz=0 0 0 rpy=1.5707963267948966 0 1.5707963267948966
- added joint robotiq_85_base_joint: type fixed, parent tool0, child robotiq_85_base_link, origin xyz=0 0 0 rpy=1.570795 -1.570795 0
- added joint robotiq_85_left_finger_joint: type continuous, parent robotiq_85_left_knuckle_link, child robotiq_85_left_finger_link, origin xyz=-0.00408552455 -0.03148604435 0.0 rpy=0 0 0
- added joint robotiq_85_left_finger_tip_joint: type continuous, parent robotiq_85_left_inner_knuckle_link, child robotiq_85_left_finger_tip_link, origin xyz=0.04303959807 -0.03759940821 0.0 rpy=0.0 0.0 0.0, axis 0 0 1, limit lower=-3.14 upper=3.14 effort=0.1 velocity=100.0, mimic joint=robotiq_85_left_knuckle_joint multiplier=-1
- added joint robotiq_85_left_inner_knuckle_joint: type continuous, parent robotiq_85_base_link, child robotiq_85_left_inner_knuckle_link, origin xyz=0.06142 0.0127 0 rpy=3.14159 0.0 0.0, axis 0 0 1, limit lower=-3.14 upper=3.14 effort=0.1 velocity=100.0, mimic joint=robotiq_85_left_knuckle_joint offset=0
- added joint robotiq_85_left_knuckle_joint: type revolute, parent robotiq_85_base_link, child robotiq_85_left_knuckle_link, origin xyz=0.05490451627 0.03060114443 0.0 rpy=3.14159 0.0 0.0, axis 0 0 1, limit lower=0.0 upper=0.804 effort=1000 velocity=2.0
- added joint robotiq_85_right_finger_joint: type continuous, parent robotiq_85_right_knuckle_link, child robotiq_85_right_finger_link, origin xyz=-0.00408552455 -0.03148604435 0.0 rpy=0 0 0
- added joint robotiq_85_right_finger_tip_joint: type continuous, parent robotiq_85_right_inner_knuckle_link, child robotiq_85_right_finger_tip_link, origin xyz=0.04303959807 -0.03759940821  0.0 rpy=0.0 0.0 0.0, axis 0 0 1, limit lower=-3.14 upper=3.14 effort=0.1 velocity=100.0, mimic joint=robotiq_85_left_knuckle_joint multiplier=-1
- added joint robotiq_85_right_inner_knuckle_joint: type continuous, parent robotiq_85_base_link, child robotiq_85_right_inner_knuckle_link, origin xyz=0.06142 -0.0127 0 rpy=0 0 0, axis 0 0 1, limit lower=-3.14 upper=3.14 effort=0.1 velocity=100.0, mimic joint=robotiq_85_left_knuckle_joint offset=0
- added joint robotiq_85_right_knuckle_joint: type continuous, parent robotiq_85_base_link, child robotiq_85_right_knuckle_link, origin xyz=0.05490451627 -0.03060114443 0.0 rpy=0.0 0.0 0.0, axis 0 0 1, limit lower=-3.14 upper=3.14 effort=1000 velocity=100.0, mimic joint=robotiq_85_left_knuckle_joint
- added joint shoulder_lift_joint: type revolute, parent shoulder_link, child upper_arm_link, origin xyz=0 0 0 rpy=1.570796327 0 0, axis 0 0 1, limit lower=-6.283185307179586 upper=6.283185307179586 effort=56.0 velocity=3.141592653589793
- added joint shoulder_pan_joint: type revolute, parent base_link_inertia, child shoulder_link, origin xyz=0 0 0.15185 rpy=0 0 0, axis 0 0 1, limit lower=-6.283185307179586 upper=6.283185307179586 effort=56.0 velocity=3.141592653589793
- added joint world_joint: type fixed, parent robot_common, child base_link, origin xyz=0.0 -0.15 0.0 rpy=0.0 0 0.0
- added joint wrist_1_joint: type revolute, parent forearm_link, child wrist_1_link, origin xyz=-0.2132 0 0.13105 rpy=0 0 0, axis 0 0 1, limit lower=-6.283185307179586 upper=6.283185307179586 effort=12.0 velocity=6.283185307179586
- added joint wrist_2_joint: type revolute, parent wrist_1_link, child wrist_2_link, origin xyz=0 -0.08535 -1.750557762378351e-11 rpy=1.570796327 0 0, axis 0 0 1, limit lower=-6.283185307179586 upper=6.283185307179586 effort=12.0 velocity=6.283185307179586
- added joint wrist_3-flange: type fixed, parent wrist_3_link, child flange, origin xyz=0 0 0 rpy=0 -1.5707963267948966 -1.5707963267948966
- added joint wrist_3_joint: type revolute, parent wrist_2_link, child wrist_3_link, origin xyz=0 0.0921 -1.8890025766262e-11 rpy=1.570796326589793 3.141592653589793 3.141592653589793, axis 0 0 1, limit lower=-6.283185307179586 upper=6.283185307179586 effort=12.0 velocity=6.283185307179586
- joint robot_common_ur3e_pedestal_joint: origin xyz=0.0 0.0 -0.38 rpy=0.0 0.0 0.0 -> xyz=0.0 -0.15 -0.38 rpy=0.0 0 0

File: evd_ros_backend/evd_ros_tasks/description/environment.urdf.xacro (robot description, xacro)
@@ -67,5 +67,5 @@
     <parent link="env_base" />
     <child link="blade_conveyor_link" />
-    <origin xyz="-0.28 0.32 0.3" rpy="0.0 0.0 0.0" />
+    <origin xyz="-0.85 -0.25 -0.75" rpy="0.0 0.0 1.5707963" />
   </joint>
   <!-- Blade Feeder -->
@@ -88,5 +88,5 @@
     <parent link="env_base" />
     <child link="blade_feeder_link" />
-    <origin xyz="-0.28 0.32 0.3" rpy="0.0 0.0 0.0" />
+    <origin xyz="-0.85 -0.25 -0.75" rpy="0.0 0.0 1.5707963" />
   </joint>
   <!-- Assembly Jig -->
@@ -109,5 +109,5 @@
     <parent link="env_base" />
     <child link="assembly_jig_link" />
-    <origin xyz="-0.28 0.32 0.3" rpy="0.0 0.0 0.0" />
+    <origin xyz="0.2 0.28 0.14" rpy="0.0 1.5707963 1.5707963" />
   </joint>
   <!-- Knife Feeder -->
@@ -130,5 +130,5 @@
     <parent link="env_base" />
     <child link="knife_feeder_link" />
-    <origin xyz="-0.28 0.32 0.3" rpy="0.0 0.0 0.0" />
+    <origin xyz="0.85 -0.25 -0.75" rpy="0.0 0.0 -1.5707963" />
   </joint>
   <!-- Knife Conveyor -->
@@ -151,5 +151,5 @@
     <parent link="env_base" />
     <child link="knife_conveyor_link" />
-    <origin xyz="-0.28 0.32 0.3" rpy="0.0 0.0 0.0" />
+    <origin xyz="0.85 -0.25 -0.75" rpy="0.0 0.0 -1.5707963" />
   </joint>
 </robot>

File: evd_ros_backend/evd_ros_tasks/description/full_task.urdf.xacro (robot description, xacro)
@@ -12,5 +12,5 @@
     <parent link="world"/>
     <child link="robot_common"/>
-    <origin xyz="0.0 0.0 0.0" rpy="0.0 0.0 0.0" />
+    <origin xyz="0.0 0 0.0" rpy="0.0 0.0 0.0" />
   </joint>
   <!-- Environment -->

File: evd_ros_backend/evd_ros_tasks/description/ur3e_single.urdf.xacro (robot description, xacro)
@@ -7,32 +7,4 @@
 	<!-- robot_common -->
 	<link name="robot_common" />
-	<!-- UR3e Physical -->
-	<xacro:include filename="$(find ur_description)/urdf/inc/ur3e_macro.xacro" />
-	<joint name="physical_common_joint" type="fixed">
-		<parent link="robot_common" />
-		<child link = "physical_base_link" />
-		<origin xyz="0.0 -0.15 0.0" rpy="0.0 0.0 0.0" />
-	</joint>
-	<xacro:ur3e_robot prefix="physical_"
-  />
-	<!-- Robotiq 85 Physical -->
-	<xacro:include filename="$(find robotiq_85_description)/urdf/robotiq_85_gripper.urdf.xacro" />
-	<xacro:robotiq_85_gripper prefix="physical_" parent="physical_tool0">
-		<origin xyz="0 0 0" rpy="${pi/2} -${pi/2} 0" />
-	</xacro:robotiq_85_gripper>
-  <!-- UR3e Simulated -->
-	<xacro:include filename="$(find ur_description)/urdf/inc/ur3e_macro.xacro" />
-	<joint name="simulated_common_joint" type="fixed">
-		<parent link="robot_common" />
-		<child link = "simulated_base_link" />
-		<origin xyz="0.0 -0.15 0.0" rpy="0.0 0.0 0.0" />
-	</joint>
-	<xacro:ur3e_robot prefix="simulated_"
-  />
-  <!-- Robotiq 85 Simulated -->
-	<xacro:include filename="$(find robotiq_85_description)/urdf/robotiq_85_gripper.urdf.xacro" />
-	<xacro:robotiq_85_gripper prefix="simulated_" parent="simulated_tool0">
-		<origin xyz="0 0 0" rpy="${pi/2} -${pi/2} 0" />
-	</xacro:robotiq_85_gripper>
 	<!-- UR3e Planner -->
 	<xacro:include filename="$(find ur_description)/urdf/inc/ur3e_macro.xacro" />
@@ -43,5 +15,5 @@
 	</joint>
 	<xacro:ur3e_robot prefix="planner_"
-  />
+  	/>
 	<!-- Robotiq 85 Planner -->
 	<xacro:include filename="$(find robotiq_85_description)/urdf/robotiq_85_gripper.urdf.xacro" />

Commit message: fixing model and creating workcell registration

File: evd_ros_backend/evd_ros_tasks/config/pybullet/environment.urdf (robot description, URDF)
Before this commit: robot environment, 8 links, 7 joints
Links:
- link 3d_printer_link: geometry visual mesh filename=./environment/visual/3d_printer.stl
- link table_link: geometry visual mesh filename=./environment/visual/table.stl

File: evd_ros_backend/evd_ros_tasks/config/pybullet/robot.urdf (robot description, URDF)
Before this commit: robot robot, 22 links, 21 joints
Links:
- link ur3e_pedestal_link: geometry visual mesh filename=package://evd_ros_tasks/description/meshes/visual/pedestal.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

File: evd_ros_backend/evd_ros_tasks/description/environment.urdf.xacro (robot description, xacro)
@@ -11,5 +11,5 @@
       <origin rpy="0 0 0" xyz="0 0 0"/>
       <geometry>
-        <mesh filename="package://evd_ros_tasks/description/meshes/visual/Table.stl"/>
+        <mesh filename="package://evd_ros_tasks/description/meshes/visual/table.stl"/>
       </geometry>
       <material name="visual_env_mesh"/>
@@ -18,5 +18,5 @@
       <origin rpy="0 0 0" xyz="0 0 0"/>
       <geometry>
-        <mesh filename="package://evd_ros_tasks/description/meshes/collision/Table.stl"/>
+        <mesh filename="package://evd_ros_tasks/description/meshes/collision/table.stl"/>
       </geometry>
     </collision>
@@ -32,5 +32,5 @@
       <origin rpy="0 0 0" xyz="0 0 0"/>
       <geometry>
-        <mesh filename="package://evd_ros_tasks/description/meshes/visual/MK2-Printer.stl"/>
+        <mesh filename="package://evd_ros_tasks/description/meshes/visual/3d_printer.stl"/>
       </geometry>
       <material name="visual_env_mesh"/>
@@ -39,5 +39,5 @@
       <origin rpy="0 0 0" xyz="0 0 0"/>
       <geometry>
-        <mesh filename="package://evd_ros_tasks/description/meshes/collision/MK2-Printer.stl"/>
+        <mesh filename="package://evd_ros_tasks/description/meshes/collision/3d_printer.stl"/>
       </geometry>
     </collision>

File: evd_ros_backend/evd_ros_tasks/description/ur3e.urdf.xacro (robot description, xacro)
@@ -54,5 +54,5 @@
       <origin rpy="0 0 0" xyz="0 0 0"/>
       <geometry>
-        <mesh filename="package://evd_ros_tasks/description/meshes/visual/Pedestal.stl"/>
+        <mesh filename="package://evd_ros_tasks/description/meshes/visual/pedestal.stl"/>
       </geometry>
       <material name="visual_robot_mesh"/>
@@ -61,5 +61,5 @@
       <origin rpy="0 0 0" xyz="0 0 0"/>
       <geometry>
-        <mesh filename="package://evd_ros_tasks/description/meshes/collision/Pedestal.stl"/>
+        <mesh filename="package://evd_ros_tasks/description/meshes/collision/pedestal.stl"/>
       </geometry>
     </collision>

File: evd_ros_backend/evd_ros_tasks/description/ur3e_single.urdf.xacro (robot description, xacro)
@@ -26,5 +26,5 @@
       <origin rpy="0 0 0" xyz="0 0 0"/>
       <geometry>
-        <mesh filename="package://evd_ros_tasks/description/meshes/visual/Pedestal.stl"/>
+        <mesh filename="package://evd_ros_tasks/description/meshes/visual/pedestal.stl"/>
       </geometry>
       <material name="visual_robot_mesh"/>
@@ -33,5 +33,5 @@
       <origin rpy="0 0 0" xyz="0 0 0"/>
       <geometry>
-        <mesh filename="package://evd_ros_tasks/description/meshes/collision/Pedestal.stl"/>
+        <mesh filename="package://evd_ros_tasks/description/meshes/collision/pedestal.stl"/>
       </geometry>
     </collision>
