Commit message: mass is removed from all objects. joint control is static instead of physics based. I know how collision meshes work now - just need to pack them

File: evd_ros_backend/evd_ros_tasks/config/pybullet/empty.urdf (robot description, URDF)
Before this commit: robot robot_name, 1 links, 0 joints
Links:
- link link_name: geometry 

File: evd_ros_backend/evd_ros_tasks/config/pybullet/robot_n_mass.urdf (robot description, URDF)
Before this commit: robot robot, 22 links, 21 joints
Links:
- link base_link_inertia: mass 2.0 -> 0; geometry collision mesh filename=./robot/collision/base.stl
- link forearm_link: mass 1.26 -> 0; geometry collision mesh filename=./robot/collision/forearm.stl
- link robotiq_85_base_link: mass 0.636951 -> 0; geometry collision mesh filename=./robot/collision/robotiq_85_base_link.stl
- link robotiq_85_left_finger_link: mass 0.027309 -> 0; geometry collision mesh filename=./robot/collision/robotiq_85_finger_link.stl
- link robotiq_85_left_finger_tip_link: mass 0.019555 -> 0; geometry collision mesh filename=./robot/collision/robotiq_85_finger_tip_link.stl
- link robotiq_85_left_inner_knuckle_link: mass 0.029951 -> 0; geometry collision mesh filename=./robot/collision/robotiq_85_inner_knuckle_link.stl
- link robotiq_85_left_knuckle_link: mass 0.018491 -> 0; geometry collision mesh filename=./robot/collision/robotiq_85_knuckle_link.stl
- link robotiq_85_right_finger_link: mass 0.027309 -> 0; geometry collision mesh filename=./robot/collision/robotiq_85_finger_link.stl
- link robotiq_85_right_finger_tip_link: mass 0.019555 -> 0; geometry collision mesh filename=./robot/collision/robotiq_85_finger_tip_link.stl
- link robotiq_85_right_inner_knuckle_link: mass 0.029951 -> 0; geometry collision mesh filename=./robot/collision/robotiq_85_inner_knuckle_link.stl
- link robotiq_85_right_knuckle_link: mass 0.018491 -> 0; geometry collision mesh filename=./robot/collision/robotiq_85_knuckle_link.stl
- link shoulder_link: mass 2.0 -> 0; geometry collision mesh filename=./robot/collision/shoulder.stl
- link upper_arm_link: mass 3.42 -> 0; geometry collision mesh filename=./robot/collision/upperarm.stl
- link ur3e_pedestal_link: mass None -> 0; geometry collision mesh filename=./environment/collision/pedestal.stl
- link wrist_1_link: mass 0.8 -> 0; geometry collision mesh filename=./robot/collision/wrist1.stl
- link wrist_2_link: mass 0.8 -> 0; geometry collision mesh filename=./robot/collision/wrist2.stl
- link wrist_3_link: mass 0.35 -> 0; geometry collision mesh filename=./robot/collision/wrist3.stl
