Commit message: updating lively config since it seems it was acting weird before + adding gripper link to urdf

File: evd_ros_backend/evd_ros_tasks/config/pybullet/robot_n_mass.urdf (robot description, URDF)
Before this commit: robot robot, 22 links, 21 joints
Links:
- added link tool0_endpoint; visual sphere radius=0.025
Joints:
- added joint tool0_to_tool0_endpoint: type fixed, parent tool0, child tool0_endpoint, origin xyz=0.0 0.0 0.15 rpy=0.0 0 0

File: evd_ros_backend/evd_ros_tasks/config/pybullet/robot_w_mass.urdf (robot description, URDF)
Before this commit: robot robot, 22 links, 21 joints
Links:
- added link tool0_endpoint; visual sphere radius=0.025
Joints:
- added joint tool0_to_tool0_endpoint: type fixed, parent tool0, child tool0_endpoint, origin xyz=0.0 0.0 0.15 rpy=0.0 0 0

File: evd_ros_backend/evd_ros_tasks/description/ur3e.urdf.xacro (robot description, xacro)
@@ -21,4 +21,17 @@
 		<origin xyz="0 0 0" rpy="${pi/2} -${pi/2} 0" />
 	</xacro:robotiq_85_gripper>
+	<link name="physical_tool0_endpoint" type="fixed">
+    <visual>
+      <origin rpy="0 0 0" xyz="0 0 0"/>
+      <geometry>
+        <sphere radius="0.025"/>
+      </geometry>
+    </visual>
+  </link>
+  <joint name="physical_tool0_to_tool0_endpoint" type="fixed">
+    <parent link="physical_tool0"/>
+    <child link="physical_tool0_endpoint"/>
+    <origin rpy="0.0 0 0" xyz="0.0 0.0 0.15"/>
+  </joint>
   <!-- UR3e Simulated -->
 	<xacro:include filename="$(find ur_description)/urdf/inc/ur3e_macro.xacro" />
@@ -35,4 +48,17 @@
 		<origin xyz="0 0 0" rpy="${pi/2} -${pi/2} 0" />
 	</xacro:robotiq_85_gripper>
+	<link name="simulated_tool0_endpoint" type="fixed">
+    <visual>
+      <origin rpy="0 0 0" xyz="0 0 0"/>
+      <geometry>
+        <sphere radius="0.025"/>
+      </geometry>
+    </visual>
+  </link>
+  <joint name="simulated_tool0_to_tool0_endpoint" type="fixed">
+    <parent link="simulated_tool0"/>
+    <child link="simulated_tool0_endpoint"/>
+    <origin rpy="0.0 0 0" xyz="0.0 0.0 0.15"/>
+  </joint>
 	<!-- UR3e Planner -->
 	<xacro:include filename="$(find ur_description)/urdf/inc/ur3e_macro.xacro" />
@@ -49,4 +75,17 @@
 		<origin xyz="0 0 0" rpy="${pi/2} -${pi/2} 0" />
 	</xacro:robotiq_85_gripper>
+	<link name="planner_tool0_endpoint" type="fixed">
+    <visual>
+      <origin rpy="0 0 0" xyz="0 0 0"/>
+      <geometry>
+        <sphere radius="0.025"/>
+      </geometry>
+    </visual>
+  </link>
+  <joint name="planner_tool0_to_tool0_endpoint" type="fixed">
+    <parent link="planner_tool0"/>
+    <child link="planner_tool0_endpoint"/>
+    <origin rpy="0.0 0 0" xyz="0.0 0.0 0.15"/>
+  </joint>
 	<!-- Robot Pedestal -->
   <link name="ur3e_pedestal_link" type="fixed" >

File: evd_ros_backend/evd_ros_tasks/description/ur3e_only.urdf.xacro (robot description, xacro)
@@ -20,3 +20,16 @@
 		<origin xyz="0 0 0" rpy="${pi/2} -${pi/2} 0" />
 	</xacro:robotiq_85_gripper>
+	<link name="planner_tool0_endpoint" type="fixed">
+    <visual>
+      <origin rpy="0 0 0" xyz="0 0 0"/>
+      <geometry>
+        <sphere radius="0.025"/>
+      </geometry>
+    </visual>
+  </link>
+  <joint name="planner_tool0_to_tool0_endpoint" type="fixed">
+    <parent link="planner_tool0"/>
+    <child link="planner_tool0_endpoint"/>
+    <origin rpy="0.0 0 0" xyz="0.0 0.0 0.15"/>
+  </joint>
 </robot>

File: evd_ros_backend/evd_ros_tasks/description/ur3e_single.urdf.xacro (robot description, xacro)
@@ -21,4 +21,17 @@
 		<origin xyz="0 0 0" rpy="${pi/2} -${pi/2} 0" />
 	</xacro:robotiq_85_gripper>
+	<link name="planner_tool0_endpoint" type="fixed">
+    <visual>
+      <origin rpy="0 0 0" xyz="0 0 0"/>
+      <geometry>
+        <sphere radius="0.025"/>
+      </geometry>
+    </visual>
+  </link>
+  <joint name="planner_tool0_to_tool0_endpoint" type="fixed">
+    <parent link="planner_tool0"/>
+    <child link="planner_tool0_endpoint"/>
+    <origin rpy="0.0 0 0" xyz="0.0 0.0 0.15"/>
+  </joint>
 	<!-- Robot Pedestal -->
   <link name="ur3e_pedestal_link" type="fixed" >
