Commit message: restructured tasks to better standardize task package with traditional ros package structure

File: evd_ros_backend/evd_ros_tasks/description/3d_printer_machine_tending.urdf.xacro (robot description, xacro)
@@ -25,5 +25,5 @@
       <origin rpy="0 0 0" xyz="0 0 0"/>
       <geometry>
-        <mesh filename="package://evd_ros_tasks/tasks/3d_printer_machine_tending/models/Table/Table.stl"/>
+        <mesh filename="package://evd_ros_tasks/description/3d_printer_machine_tending/visual_meshes/Table.stl"/>
       </geometry>
       <material name="visual_app_mesh"/>
@@ -32,5 +32,5 @@
       <origin rpy="0 0 0" xyz="0 0 0"/>
       <geometry>
-        <mesh filename="package://evd_ros_tasks/tasks/3d_printer_machine_tending/collision_meshes/Table.stl"/>
+        <mesh filename="package://evd_ros_tasks/description/3d_printer_machine_tending/collision_meshes/Table.stl"/>
       </geometry>
     </collision>
@@ -46,5 +46,5 @@
       <origin rpy="0 0 0" xyz="0 0 0"/>
       <geometry>
-        <mesh filename="package://evd_ros_tasks/tasks/3d_printer_machine_tending/models/MK2-Printer/MK2-Printer.stl"/>
+        <mesh filename="package://evd_ros_tasks/description/3d_printer_machine_tending/visual_meshes/MK2-Printer.stl"/>
       </geometry>
       <material name="visual_app_mesh"/>
@@ -53,5 +53,5 @@
       <origin rpy="0 0 0" xyz="0 0 0"/>
       <geometry>
-        <mesh filename="package://evd_ros_tasks/tasks/3d_printer_machine_tending/collision_meshes/MK2-Printer.stl"/>
+        <mesh filename="package://evd_ros_tasks/description/3d_printer_machine_tending/collision_meshes/MK2-Printer.stl"/>
       </geometry>
     </collision>
@@ -67,5 +67,5 @@
       <origin rpy="0 0 0" xyz="0 0 0"/>
       <geometry>
-        <mesh filename="package://evd_ros_tasks/tasks/3d_printer_machine_tending/models/Box/Box.stl"/>
+        <mesh filename="package://evd_ros_tasks/description/3d_printer_machine_tending/visual_meshes/Box.stl"/>
       </geometry>
       <material name="visual_app_mesh"/>
@@ -74,5 +74,5 @@
       <origin rpy="0 0 0" xyz="0 0 0"/>
       <geometry>
-        <mesh filename="package://evd_ros_tasks/tasks/3d_printer_machine_tending/collision_meshes/Box.stl"/>
+        <mesh filename="package://evd_ros_tasks/description/3d_printer_machine_tending/collision_meshes/Box.stl"/>
       </geometry>
     </collision>
@@ -88,5 +88,5 @@
       <origin rpy="0 0 0" xyz="0 0 0"/>
       <geometry>
-        <mesh filename="package://evd_ros_tasks/tasks/3d_printer_machine_tending/models/ur3e-Pedestal/Pedestal.stl"/>
+        <mesh filename="package://evd_ros_tasks/description/3d_printer_machine_tending/visual_meshes/Pedestal.stl"/>
       </geometry>
       <material name="visual_app_mesh"/>
@@ -95,5 +95,5 @@
       <origin rpy="0 0 0" xyz="0 0 0"/>
       <geometry>
-        <mesh filename="package://evd_ros_tasks/tasks/3d_printer_machine_tending/collision_meshes/Pedestal.stl"/>
+        <mesh filename="package://evd_ros_tasks/description/3d_printer_machine_tending/collision_meshes/Pedestal.stl"/>
       </geometry>
     </collision>

Commit message: Simulation and /tf connection

File: evd_ros_backend/evd_ros_tasks/description/3d_printer_machine_tending.urdf.xacro (robot description, xacro)
@@ -39,5 +39,5 @@
     <parent link="app" />
     <child link="table_link" />
-    <origin xyz="0.0 0.36 -0.37" rpy="0.0 0.0 0.0" />
+    <origin xyz="1.0 0.36 -0.37" rpy="0.0 0.0 0.0" />
   </joint>
   <!-- 3D Printer -->

Commit message: debugging

File: evd_ros_backend/evd_ros_tasks/description/3d_printer_machine_tending.urdf.xacro (robot description, xacro)
@@ -39,5 +39,5 @@
     <parent link="app" />
     <child link="table_link" />
-    <origin xyz="1.0 0.36 -0.37" rpy="0.0 0.0 0.0" />
+    <origin xyz="0.0 0.36 -0.37" rpy="0.0 0.0 0.0" />
   </joint>
   <!-- 3D Printer -->
