Commit message: joint interpolation in trace processor generally working + working on URDFs for collision_meshes

File: evd_ros_backend/evd_ros_tasks/config/pybullet/collision_mesh_urdf/3d_printer.stl.urdf (robot description, URDF)
Before this commit: robot 3d_printer, 1 links, 0 joints
Links:
- removed link 3d_printer
- added link collision_mesh_3d_printer, mass 0; collision mesh filename=./environment/3d_printer.stl; visual mesh filename=./environment/3d_printer.stl

File: evd_ros_backend/evd_ros_tasks/config/pybullet/collision_mesh_urdf/assembly_jig.stl.urdf (robot description, URDF)
Before this commit: robot assembly_jig, 1 links, 0 joints
Links:
- removed link assembly_jig
- added link collision_mesh_assembly_jig, mass 0; collision mesh filename=./environment/assembly_jig.stl; visual mesh filename=./environment/assembly_jig.stl

File: evd_ros_backend/evd_ros_tasks/config/pybullet/collision_mesh_urdf/blade_feeder.stl.urdf (robot description, URDF)
Before this commit: robot blade_feeder, 1 links, 0 joints
Links:
- removed link blade_feeder
- added link collision_mesh_blade_feeder, mass 0; collision mesh filename=./environment/blade_feeder.stl; visual mesh filename=./environment/blade_feeder.stl

File: evd_ros_backend/evd_ros_tasks/config/pybullet/collision_mesh_urdf/box.stl.urdf (robot description, URDF)
Before this commit: robot box, 1 links, 0 joints
Links:
- removed link box
- added link collision_mesh_box, mass 0; collision mesh filename=./environment/box.stl; visual mesh filename=./environment/box.stl

File: evd_ros_backend/evd_ros_tasks/config/pybullet/collision_mesh_urdf/conveyor.stl.urdf (robot description, URDF)
Before this commit: robot conveyor, 1 links, 0 joints
Links:
- removed link conveyor
- added link collision_mesh_conveyor, mass 0; collision mesh filename=./environment/conveyor.stl; visual mesh filename=./environment/conveyor.stl

File: evd_ros_backend/evd_ros_tasks/config/pybullet/collision_mesh_urdf/knife_feeder.stl.urdf (robot description, URDF)
Before this commit: robot knife_feeder, 1 links, 0 joints
Links:
- removed link knife_feeder
- added link collision_mesh_knife_feeder, mass 0; collision mesh filename=./environment/knife_feeder.stl; visual mesh filename=./environment/knife_feeder.stl

File: evd_ros_backend/evd_ros_tasks/config/pybullet/collision_mesh_urdf/pedestal.stl.urdf (robot description, URDF)
Before this commit: robot pedestal, 1 links, 0 joints
Links:
- removed link pedestal
- added link collision_mesh_pedestal, mass 0; collision mesh filename=./environment/pedestal.stl; visual mesh filename=./environment/pedestal.stl

File: evd_ros_backend/evd_ros_tasks/config/pybullet/collision_mesh_urdf/table.stl.urdf (robot description, URDF)
Before this commit: robot table, 1 links, 0 joints
Links:
- removed link table
- added link collision_mesh_table, mass 0; collision mesh filename=./environment/table.stl; visual mesh filename=./environment/table.stl
