Commit message: proving each collision URDF loads properly + fixing workcell to register machine inputs and outputs with correct format

File: evd_ros_backend/evd_ros_tasks/config/pybullet/collision_mesh_urdfs/3d_printer.stl.urdf (robot description, URDF)
Before this commit: robot pedestal, 1 links, 0 joints
Links:
- removed link collision_mesh_pedestal
- added link collision_mesh_3d_printer, mass 0; collision mesh filename=../environment/collision/3d_printer.stl

File: evd_ros_backend/evd_ros_tasks/config/pybullet/collision_mesh_urdfs/assembly_jig.stl.urdf (robot description, URDF)
Before this commit: robot table, 1 links, 0 joints
Links:
- removed link collision_mesh_table
- added link collision_mesh_assembly_jig, mass 0; collision mesh filename=../environment/collision/assembly_jig.stl

File: evd_ros_backend/evd_ros_tasks/config/pybullet/collision_mesh_urdfs/blade_feeder.stl.urdf (robot description, URDF)
Before this commit: robot knife_feeder, 1 links, 0 joints
Links:
- removed link collision_mesh_knife_feeder
- added link collision_mesh_blade_feeder, mass 0; collision mesh filename=../environment/collision/blade_feeder.stl

File: evd_ros_backend/evd_ros_tasks/config/pybullet/collision_mesh_urdfs/box.stl.urdf (robot description, URDF)
Before this commit: robot assembly_jig, 1 links, 0 joints
Links:
- removed link collision_mesh_assembly_jig
- added link collision_mesh_box, mass 0; collision mesh filename=../environment/collision/box.stl

File: evd_ros_backend/evd_ros_tasks/config/pybullet/collision_mesh_urdfs/conveyor.stl.urdf (robot description, URDF)
Before this commit: robot conveyor, 1 links, 0 joints
Links:
- link collision_mesh_conveyor: geometry collision mesh filename=../environment/collision/conveyor.stl

File: evd_ros_backend/evd_ros_tasks/config/pybullet/collision_mesh_urdfs/knife_feeder.stl.urdf (robot description, URDF)
Before this commit: robot box, 1 links, 0 joints
Links:
- removed link collision_mesh_box
- added link collision_mesh_knife_feeder, mass 0; collision mesh filename=../environment/collision/knife_feeder.stl

File: evd_ros_backend/evd_ros_tasks/config/pybullet/collision_mesh_urdfs/pedestal.stl.urdf (robot description, URDF)
Before this commit: robot 3d_printer, 1 links, 0 joints
Links:
- removed link collision_mesh_3d_printer
- added link collision_mesh_pedestal, mass 0; collision mesh filename=../environment/collision/pedestal.stl

File: evd_ros_backend/evd_ros_tasks/config/pybullet/collision_mesh_urdfs/table.stl.urdf (robot description, URDF)
Before this commit: robot blade_feeder, 1 links, 0 joints
Links:
- removed link collision_mesh_blade_feeder
- added link collision_mesh_table, mass 0; collision mesh filename=../environment/collision/table.stl

File: evd_ros_backend/evd_ros_tasks/config/pybullet/environment.urdf (robot description, URDF)
Before this commit: robot environment, 8 links, 7 joints
Links:
- link 3d_printer_link: mass None -> 0; geometry collision mesh filename=./environment/collision/3d_printer.stl
- link assembly_jig_link: mass None -> 0; geometry collision mesh filename=./environment/collision/assembly_jig.stl
- link blade_conveyor_link: mass None -> 0; geometry collision mesh filename=./environment/collision/conveyor.stl
- link blade_feeder_link: mass None -> 0; geometry collision mesh filename=./environment/collision/blade_feeder.stl
- link knife_conveyor_link: mass None -> 0; geometry collision mesh filename=./environment/collision/conveyor.stl
- link knife_feeder_link: mass None -> 0; geometry collision mesh filename=./environment/collision/knife_feeder.stl
- link table_link: mass None -> 0; geometry collision mesh filename=./environment/collision/table.stl

File: evd_ros_backend/evd_ros_tasks/config/pybullet/robot.urdf (robot description, URDF)
Before this commit: robot robot, 22 links, 21 joints
Links:
- link ur3e_pedestal_link: geometry visual mesh filename=./environment/visual/pedestal.stl
